File: punching_pcb/schematic.brd (EAGLE design)
At the start: 135.9 x 46.7 mm, 23 parts, among them IC1 ATMEGA328PB-AN, IC2 7805TV, J11 POWER_JACK, J3 CON_TERMINAL_BLOCK_02-5MM, J4 CON_TERMINAL_BLOCK_02-5MM, J5 CON_TERMINAL_BLOCK_02-5MM

Commit message: dd the PCB designs backup
Parts:
- removed J11: POWER_JACK, SparkFun-Connectors:POWER_JACK_PTH
- added J1: 5.5x2.1mm Barrel, SparkFun-Connectors:POWER_JACK_SMD
Connections:
- net GND: now also J1.P$4; no longer J11.GND
- net N$4: now also J1.VIN0; no longer J11.PWR
Routing:
- net GND: track 252.5 -> 258.9 mm, vias 4 -> 5
- net N$4: track 41.5 -> 44.2 mm, vias 0 -> 1
Changed lines of the file:
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@@
 <attribute name="NAME" x="57.658" y="16.002" size="1.27" layer="26" rot="MR90"/>
-</element>
-<element name="J11" library="SparkFun-Connectors" package="POWER_JACK_PTH" value="POWER_JACK" x="7.62" y="1.27" smashed="yes">
-<attribute name="NAME" x="6.2484" y="3.0988" size="0.6096" layer="25" font="vector" ratio="20"/>
-<attribute name="PROD_ID" value="CONN-08197" x="27.94" y="0" size="1.778" layer="27" display="off"/>
-<attribute name="VALUE" x="5.8674" y="2.0828" size="0.6096" layer="27" font="vector" ratio="20"/>
 </element>
 <element name="J3" library="dp_devices.v6" package="TERMINAL_BLOCK_2P_5" value="CON_TERMINAL_BLOCK_02-5MM" x="128.27" y="5.08" smashed="yes">
@@
 <attribute name="NAME" x="64.77" y="1.905" size="0.6096" layer="25" rot="R180"/>
 <attribute name="VALUE" x="64.77" y="3.81" size="0.6096" layer="27" rot="R180"/>
+</element>
+<element name="J1" library="SparkFun-Connectors" package="POWER_JACK_SMD" value="5.5x2.1mm Barrel" x="2.54" y="6.35" smashed="yes">
+<attribute name="NAME" x="6.6802" y="9.144" size="0.6096" layer="25" font="vector" ratio="20"/>
+<attribute name="PROD_ID" value="CONN-08106" x="2.54" y="6.35" size="1.778" layer="27" display="off"/>
+<attribute name="SF_ID" value="PRT-12748" x="2.54" y="6.35" size="1.778" layer="27" display="off"/>
+<attribute name="VALUE" x="6.35" y="3.048" size="0.6096" layer="27" font="vector" ratio="20"/>
 </element>
 </elements>
@@
 <contactref element="SD-FORMAT" pad="3"/>
 <contactref element="IC2" pad="2"/>
-<contactref element="J11" pad="GND"/>
 <contactref element="C1" pad="2"/>
 <contactref element="12V-INPUT" pad="2"/>
@@
 <contactref element="DEGBUG" pad="4"/>
 <contactref element="SD-CARD-HOLDER" pad="6"/>
-<wire x1="7.62" y1="8.97" x2="2.62" y2="13.97" width="2.032" layer="16"/>
-<wire x1="2.62" y1="13.97" x2="2.54" y2="13.97" width="2.032" layer="16"/>
-<wire x1="2.032" y1="14.478" x2="2.54" y2="13.97" width="2.032" layer="16"/>
-<wire x1="7.62" y1="8.97" x2="14.558" y2="2.032" width="2.032" layer="16"/>
 <wire x1="14.558" y1="2.032" x2="19.05" y2="2.032" width="2.032" layer="16"/>
 <wire x1="35.56" y1="8.89" x2="35.56" y2="3.81" width="2.032" layer="16"/>
@@
 <wire x1="53.3" y1="7.66" x2="48.26" y2="12.7" width="1.778" layer="16"/>
 <wire x1="6.8" y1="22.9" x2="2.032" y2="18.132" width="1.778" layer="16"/>
-<wire x1="2.032" y1="18.132" x2="2.032" y2="14.478" width="1.778" layer="16"/>
+<contactref element="J1" pad="P$4"/>
+<wire x1="8.64" y1="0.65" x2="13.176" y2="0.65" width="1.524" layer="1"/>
+<wire x1="13.176" y1="0.65" x2="14.558" y2="2.032" width="1.524" layer="1"/>
+<via x="14.558" y="2.032" extent="1-16" drill="0.35"/>
+<wire x1="9.906" y1="7.50731875" x2="9.906" y2="6.684" width="1.524" layer="16"/>
+<wire x1="9.906" y1="6.684" x2="14.558" y2="2.032" width="1.524" layer="16"/>
+<wire x1="2.032" y1="18.132" x2="2.032" y2="15.38131875" width="1.524" layer="16"/>
+<wire x1="2.032" y1="15.38131875" x2="9.906" y2="7.50731875" width="1.524" layer="16"/>
 </signal>
 <signal name="VCC">
@@
 </signal>
 <signal name="N$4">
-<contactref element="J11" pad="PWR"/>
 <contactref element="D6" pad="A"/>
 <contactref element="12V-INPUT" pad="1"/>
-<wire x1="7.62" y1="14.97" x2="10.43" y2="17.78" width="2.032" layer="16"/>
 <wire x1="15.24" y1="17.78" x2="17.78" y2="15.24" width="2.032" layer="16"/>
 <wire x1="17.78" y1="6.35" x2="16.51" y2="5.08" width="2.032" layer="16"/>
@@
 <wire x1="6.8" y1="27.9" x2="10.2" y2="27.9" width="1.778" layer="16"/>
 <wire x1="10.2" y1="27.9" x2="11.43" y2="26.67" width="1.778" layer="16"/>
-<wire x1="11.43" y1="18.78" x2="7.62" y2="14.97" width="1.778" layer="16"/>
-<wire x1="11.43" y1="26.67" x2="11.43" y2="18.78" width="1.778" layer="16"/>
+<wire x1="11.43" y1="18.78" x2="11.43" y2="26.67" width="1.778" layer="16"/>
+<contactref element="J1" pad="VIN0"/>
+<wire x1="2.54" y1="12.05" x2="6.35" y2="15.86" width="1.524" layer="1"/>
+<wire x1="6.35" y1="15.86" x2="6.35" y2="16.51" width="1.524" layer="1"/>
+<wire x1="6.35" y1="16.51" x2="7.62" y2="17.78" width="1.524" layer="1"/>
+<wire x1="7.62" y1="17.78" x2="10.43" y2="17.78" width="1.524" layer="1"/>
+<via x="10.43" y="17.78" extent="1-16" drill="0.35"/>
+<wire x1="10.43" y1="17.78" x2="11.43" y2="18.78" width="1.524" layer="16"/>
 </signal>
 <signal name="N$5">
